File: Trx_antena_pcb/Radio.sch (KiCad schematic (older format))
At the start: 29 parts, among them U1 CC2520, U2 CC2591, X1 32MHz

Commit message: "Segundas correcciones. Documentacion"
Connections:
- net VREG_EN: now also R2.2, U1.26 (VREG_EN)
Other:
- moved on the sheet: R2
Changed lines of the file:
@@
 EESchema Schematic File Version 2
-LIBS:dongle
-LIBS:ubertooth-symbols
-LIBS:Ej2-cache
-LIBS:juanvmont-cache
 LIBS:device
 LIBS:Trx_antena_pcb-cache
@@
 $Descr A4 11693 8268
 encoding utf-8
-Sheet 3 3
-Title ""
-Date ""
-Rev ""
-Comp ""
-Comment1 ""
-Comment2 ""
-Comment3 ""
-Comment4 ""
+Sheet 2 2
+Title "Poncho EDU-CIAA-NXP RF 2.4GHz Antena PCB"
+Date "2016-12-02"
+Rev "1.0"
+Comp "Proyecto CIAA - COMPUTADORA INDUSTRIAL ABIERTA ARGENTINA"
+Comment1 "https://github.com/ciaa/Ponchos/tree/master/modelos/doc"
+Comment2 "Basado en el template de Diego Brengi - UNLaM"
+Comment3 "Autor y Licencia del poncho (Juan Vicente Montilla-FIUBA). Ver directorio \"doc\""
+Comment4 "https://github.com/Juanvmont/Poncho-EDU-CIAA-NXP-RF-2.4GHz-Antena-PCB.git"
 $EndDescr
 $Comp
@@
 L R R2
 U 1 1 5834A0FA
-P 1900 2450
-F 0 "R2" V 1980 2450 50  0000 C CNN
-F 1 "100K" V 1900 2450 50  0000 C CNN
-F 2 "R_0402" H 1830 2450 50  0001 C CNN
-F 3 "" H 1900 2450 50  0000 C CNN
-F 4 "RMCF0402JT1M00CT-ND" H 1900 2450 60  0001 C CNN "Digikey#"
-	1    1900 2450
+P 1900 2400
+F 0 "R2" V 1980 2400 50  0000 C CNN
+F 1 "100K" V 1900 2400 50  0000 C CNN
+F 2 "R_0402" H 1830 2400 50  0001 C CNN
+F 3 "" H 1900 2400 50  0000 C CNN
+F 4 "RMCF0402JT1M00CT-ND" H 1900 2400 60  0001 C CNN "Digikey#"
+	1    1900 2400
 	1    0    0    -1
 $EndComp
@@
 $EndComp
 NoConn ~ 6000 3500
-Text Label 2100 2600 0    60   ~ 0
+Text Label 2150 2400 0    60   ~ 0
 VREG_EN
 $Comp
@@
 Connection ~ 1450 4150
 Wire Wire Line
-	1900 2300 1900 2200
-Wire Wire Line
 	1700 2700 1700 2650
 Wire Wire Line
@@
 	1700 2350 1700 2200
 Connection ~ 1700 2200
+Text HLabel 2400 2750 0    60   Input ~ 0
+VREG_EN
+Wire Wire Line
+	1900 2250 1900 2200
+Wire Wire Line
+	1900 2550 1900 2600
+Wire Wire Line
+	1900 2600 2550 2600
+Wire Wire Line
+	2400 2750 2500 2750
+Wire Wire Line
+	2500 2750 2500 2600
+Connection ~ 2500 2600
 $EndSCHEMATC

Commit message: Completando esquematico de RF
Parts:
- added C? (x2): 1nF, C_0402, symbol C
- added C?: 2.2uF/4V, C_0402, symbol C
- added C?: 15pF, C_0402, symbol C
- added L?: 1 K, C_0402, symbol INDUCTOR
- added L?: 5.1nH, C_0402, symbol INDUCTOR
- added L?: 1.1nH, C_0402, symbol INDUCTOR
- added R?: 330, R_0402, symbol R
- added R? (x6): 0, R_0402, symbol R
- L? (x2): footprint (none) -> C_0402
- L? (x4): value 1 nF -> 1.0nH; footprint (none) -> C_0402
- L?: value 1 nF -> 1.5nH; footprint (none) -> C_0402
- R3: Digikey# RMCF0402JT1M00CT-ND -> 311-56.0KLRCT-ND
Connections:
- net +5V: now also L?.1
- net GND: now also C4.1, U1.29 (AGND), U2.14 (GND), C?.1, C?.1, C?.2, C?.2, R?.2
- net SO: now reaches U1.1 (SO)
- net SO: now also R1.1
- net GPIO0: now reaches U1.10 (GPIO0)
- net at U1.17 (RF_P): now also C7.1
- net SI: now reaches U1.2 (SI)
- net SCLK: now reaches U1.28 (SCLK)
- net CSn: now reaches U1.3 (~CS)
- net GPIO5: now reaches U1.4 (GPIO5)
- net GPIO5: now also R?.2
- net GPIO4: now reaches U1.5 (GPIO4)
- net GPIO4: now also R?.2
- net GPIO3: now reaches U1.6 (GPIO3)
- net GPIO3: now also R?.2
- net GPIO2: now reaches U1.7 (GPIO2)
- net GPIO1: now reaches U1.9 (GPIO1)
- net TL11: now reaches U2.1 (AVDD_PA1)
- net TL11: now also U2.13 (AVDD_LNA), C?.1, C?.2, C?.2, L?.1, L?.2
- net TL101: now reaches U2.10 (AVDD_PA2)
- net TL101: now also L?.1, L?.2
- net PAEN: now reaches U2.5 (PAEN)
- net PAEN: now also R?.1, R?.1, R?.1
- net EN: now reaches U2.6 (EN)
- net EN: now also R?.1, R?.1
- net HGM: now reaches U2.7 (HGM)
- net HGM: now also R?.1, R?.1
- new net: C?.1, L?.2
- new net P0.6: R?.2
- new net P2.4: R?.2
- new net P2.5: R?.2
Other:
- note added: "TLINE inductor"
- moved on the sheet: 1uF/6.3V1, C5, C6, C8, L?, R1, X1

Commit message: mattching pin tou from edu ciaa to poncho
Connections:
- net P0.6 renamed GPIO6
- net P2.4 renamed GPIO8
- net P2.5 renamed GPIO7
Changed lines of the file:
@@
 GPIO3
 Text HLabel 5200 4750 0    60   Input ~ 0
-P0.6
+GPIO6
 Text HLabel 5200 5050 0    60   Input ~ 0
-P2.5
+GPIO7
 Text HLabel 5200 5350 0    60   Input ~ 0
-P2.4
+GPIO8
 $Comp
 L C C?

Commit message: completando el esquematico
Parts:
- removed R? (x2): 0, R_0402, symbol R
- gave numbers to parts that had none: 19
- renumbered C5 to C1, C9 to C12, C10 to C13, C11 to C15, C12 to C16, C6 to C2, C2 to C3, C3 to C4, C4 to C5, C7 to C6, C1 to C7, R2 to R1, R5 to R10, R1 to R2, R4 to R9
Connections:
- net GPIO8 is gone; now on net GPIO6: R7.2
- net at 1uF/6.3V1.1, C3.2, C4.2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: now also U1.20 (AVDD1)
- net RESET: now reaches U1.25 (~RESET)

Commit message: cuarta correccion: revision2 en /doc
Parts:
- C15: Digikey# 490-1276-1-ND -> 490-5950-1-ND
- C16: Digikey# 490-1269-1-ND -> 490-5934-1-ND
Other:
- moved on the sheet: R4, R5, R6, R7, R8
Changed lines of the file:
@@
 EESchema Schematic File Version 2
-LIBS:device
+LIBS:power
 LIBS:Trx_antena_pcb-cache
 EELAYER 25 0
@@
 L GND #PWR015
 U 1 1 5830F17C
-P 6750 5050
-F 0 "#PWR015" H 6750 5050 30  0001 C CNN
-F 1 "GND" H 6750 4980 30  0001 C CNN
-F 2 "" H 6750 5050 60  0000 C CNN
-F 3 "" H 6750 5050 60  0000 C CNN
-	1    6750 5050
-	1    0    0    -1
+P 6350 4750
+F 0 "#PWR015" H 6350 4750 30  0001 C CNN
+F 1 "GND" H 6350 4680 30  0001 C CNN
+F 2 "" H 6350 4750 60  0000 C CNN
+F 3 "" H 6350 4750 60  0000 C CNN
+	1    6350 4750
+	0    1    1    0
 $EndComp
 $Comp
@@
 F 1 "6.8pF" H 9075 3300 50  0000 L CNN
 F 2 "C_0402" H 9088 3250 50  0001 C CNN
-F 3 "http://media.digikey.com/pdf/Data%20Sheets/Murata%20PDFs/Chip%20Monolithic%20Ceramic%20Caps.pdf" H 9050 3400 50  0001 C CNN
-F 4 "490-1276-1-ND" H 9050 3400 60  0001 C CNN "Digikey#"
+F 3 "http://www.murata.com/~/media/webrenewal/support/library/catalog/products/capacitor/mlcc/c02e.pdf" H 9050 3400 50  0001 C CNN
+F 4 "490-5950-1-ND" H 9050 3400 60  0001 C CNN "Digikey#"
 	1    9050 3400
 	0    -1   -1   0
@@
 F 1 "2.7pF" H 9325 3450 50  0000 L CNN
 F 2 "C_0402" H 9338 3400 50  0001 C CNN
-F 3 "http://media.digikey.com/pdf/Data%20Sheets/Murata%20PDFs/Chip%20Monolithic%20Ceramic%20Caps.pdf" H 9300 3550 50  0001 C CNN
-F 4 "490-1269-1-ND" H 9300 3550 60  0001 C CNN "Digikey#"
+F 3 "http://www.murata.com/~/media/webrenewal/support/library/catalog/products/capacitor/mlcc/c02e.pdf" H 9300 3550 50  0001 C CNN
+F 4 "490-5934-1-ND" H 9300 3550 60  0001 C CNN "Digikey#"
 	1    9300 3550
 	1    0    0    -1
@@
 L R R8
 U 1 1 584D6395
-P 6750 4800
-F 0 "R8" V 6830 4800 50  0000 C CNN
-F 1 "330" V 6750 4800 50  0000 C CNN
-F 2 "R_0402" V 6680 4800 50  0001 C CNN
-F 3 "http://www.yageo.com.tw/exep/pages/download/literatures/PYu-R_INT-thick_7.pdf" H 6750 4800 50  0001 C CNN
-F 4 "311-330JRCT-ND" H 6750 4800 60  0001 C CNN "Digikey#"
-	1    6750 4800
-	1    0    0    -1
+P 6600 4750
+F 0 "R8" V 6680 4750 50  0000 C CNN
+F 1 "330" V 6600 4750 50  0000 C CNN
+F 2 "R_0402" V 6530 4750 50  0001 C CNN
+F 3 "http://www.yageo.com.tw/exep/pages/download/literatures/PYu-R_INT-thick_7.pdf" H 6600 4750 50  0001 C CNN
+F 4 "311-330JRCT-ND" H 6600 4750 60  0001 C CNN "Digikey#"
+	1    6600 4750
+	0    1    1    0
 $EndComp
 $Comp
 L R R4
 U 1 1 584E0D86
-P 5450 4600
-F 0 "R4" V 5530 4600 50  0000 C CNN
-F 1 "0" V 5450 4600 50  0000 C CNN
-F 2 "R_0402" V 5380 4600 50  0001 C CNN
-F 3 "https://www.seielect.com/Catalog/SEI-RMCF_RMCP.pdf" H 5450 4600 50  0001 C CNN
-F 4 "RMCF0402ZT0R00CT-ND" H 5450 4600 60  0001 C CNN "Digikey#"
-	1    5450 4600
-	0    1    1    0
+P 6750 5000
+F 0 "R4" H 6750 4850 50  0000 C CNN
+F 1 "0" V 6750 5000 50  0000 C CNN
+F 2 "R_0402" V 6680 5000 50  0001 C CNN
+F 3 "https://www.seielect.com/Catalog/SEI-RMCF_RMCP.pdf" H 6750 5000 50  0001 C CNN
+F 4 "RMCF0402ZT0R00CT-ND" H 6750 5000 60  0001 C CNN "Digikey#"
+	1    6750 5000
+	1    0    0    -1
 $EndComp
 $Comp
 L R R5
 U 1 1 584E2523
-P 5450 4900
-F 0 "R5" V 5530 4900 50  0000 C CNN
-F 1 "0" V 5450 4900 50  0000 C CNN
-F 2 "R_0402" V 5380 4900 50  0001 C CNN
-F 3 "https://www.seielect.com/Catalog/SEI-RMCF_RMCP.pdf" H 5450 4900 50  0001 C CNN
-F 4 "RMCF0402ZT0R00CT-ND" H 5450 4900 60  0001 C CNN "Digikey#"
-	1    5450 4900
-	0    1    1    0
+P 6850 5000
+F 0 "R5" H 6850 4850 50  0000 C CNN
+F 1 "0" V 6850 5000 50  0000 C CNN
+F 2 "R_0402" V 6780 5000 50  0001 C CNN
+F 3 "https://www.seielect.com/Catalog/SEI-RMCF_RMCP.pdf" H 6850 5000 50  0001 C CNN
+F 4 "RMCF0402ZT0R00CT-ND" H 6850 5000 60  0001 C CNN "Digikey#"
+	1    6850 5000
+	1    0    0    -1
 $EndComp
 $Comp
 L R R6
 U 1 1 584E28F5
-P 5450 5200
-F 0 "R6" V 5530 5200 50  0000 C CNN
-F 1 "0" V 5450 5200 50  0000 C CNN
-F 2 "R_0402" V 5380 5200 50  0001 C CNN
-F 3 "https://www.seielect.com/Catalog/SEI-RMCF_RMCP.pdf" H 5450 5200 50  0001 C CNN
-F 4 "RMCF0402ZT0R00CT-ND" H 5450 5200 60  0001 C CNN "Digikey#"
-	1    5450 5200
-	0    1    1    0
+P 6950 5000
+F 0 "R6" H 6950 4850 50  0000 C CNN
+F 1 "0" V 6950 5000 50  0000 C CNN
+F 2 "R_0402" V 6880 5000 50  0001 C CNN
+F 3 "https://www.seielect.com/Catalog/SEI-RMCF_RMCP.pdf" H 6950 5000 50  0001 C CNN
+F 4 "RMCF0402ZT0R00CT-ND" H 6950 5000 60  0001 C CNN "Digikey#"
+	1    6950 5000
+	1    0    0    -1
 $EndComp
 $Comp
 L R R7
 U 1 1 584E29A9
-P 5450 5350
-F 0 "R7" V 5530 5350 50  0000 C CNN
-F 1 "0" V 5450 5350 50  0000 C CNN
-F 2 "R_0402" V 5380 5350 50  0001 C CNN
-F 3 "https://www.seielect.com/Catalog/SEI-RMCF_RMCP.pdf" H 5450 5350 50  0001 C CNN
-F 4 "RMCF0402ZT0R00CT-ND" H 5450 5350 60  0001 C CNN "Digikey#"
-	1    5450 5350
-	0    1    1    0
-$EndComp
-Text Label 5800 4600 0    60   ~ 0
-PAEN
-Text Label 5800 4900 0    60   ~ 0
-EN
-Text Label 5800 5200 0    60   ~ 0
-HGM
-Text HLabel 5200 4600 0    60   Input ~ 0
+P 7050 5000
+F 0 "R7" H 7050 4850 50  0000 C CNN
+F 1 "0" V 7050 5000 50  0000 C CNN
+F 2 "R_0402" V 6980 5000 50  0001 C CNN
+F 3 "https://www.seielect.com/Catalog/SEI-RMCF_RMCP.pdf" H 7050 5000 50  0001 C CNN
+F 4 "RMCF0402ZT0R00CT-ND" H 7050 5000 60  0001 C CNN "Digikey#"
+	1    7050 5000
+	1    0    0    -1
+$EndComp
+Text HLabel 6750 5250 3    60   Input ~ 0
 GPIO5
-Text HLabel 5200 4900 0    60   Input ~ 0
+Text HLabel 6850 5250 3    60   Input ~ 0
 GPIO4
-Text HLabel 5200 5200 0    60   Input ~ 0
+Text HLabel 6950 5250 3    60   Input ~ 0
 GPIO3
-Text HLabel 5200 5350 0    60   Input ~ 0
+Text HLabel 7050 5250 3    60   Input ~ 0
 GPIO6
 $Comp
@@
 	4950 4000 4950 4050
 Wire Wire Line
-	6750 4350 6750 4650
-Wire Wire Line
-	6850 4600 6850 4350
-Wire Wire Line
-	6950 4600 6950 4350
-Wire Wire Line
-	6750 5050 6750 4950
-Wire Wire Line
-	5800 4600 5600 4600
-Wire Wire Line
-	5800 4900 5600 4900
-Wire Wire Line
-	5800 5200 5600 5200
-Wire Wire Line
-	5700 5200 5700 5350
-Wire Wire Line
-	5700 5350 5600 5350
-Connection ~ 5700 5200
-Wire Wire Line
-	5300 4600 5200 4600
-Wire Wire Line
-	5300 4900 5200 4900
-Wire Wire Line
-	5300 5200 5200 5200
-Wire Wire Line
-	5300 5350 5200 5350
+	6750 4350 6750 4850
+Wire Wire Line
+	6950 4350 6950 4850
+Wire Wire Line
+	6350 4750 6450 4750
+Connection ~ 6950 4750
+Wire Wire Line
+	6750 5150 6750 5250
+Wire Wire Line
+	6850 5150 6850 5250
+Wire Wire Line
+	6950 5150 6950 5250
+Wire Wire Line
+	7050 5150 7050 5250
 Wire Wire Line
 	6950 2550 6950 2500
@@
 	2900 2200 2900 2000
 Connection ~ 2900 2200
+Connection ~ 6750 4750
+Wire Wire Line
+	6850 4350 6850 4850
+Wire Wire Line
+	6950 4750 7050 4750
+Wire Wire Line
+	7050 4750 7050 4850
 $EndSCHEMATC

Commit message: layout de componentes en pcbnew
Parts:
- 1uF/6.3V1, C1, C10, C11, C12, C13, C14, C15, C16, C2, C3, C4, C5, C6, C7, C8, C9, L1, L10, L2, L3, L4, L5, L6, L7, L8, L9: footprint C_0402 -> Capacitors_SMD:C_0402
- A1: footprint INV_F_ANT -> Wpan_Prints:INV_F_ANT
- R1, R10, R2, R3, R4, R5, R6, R7, R8, R9: footprint R_0402 -> Resistors_SMD:R_0402
- U1: footprint QFN50P500X500X100-28N -> Housings_DFN_QFN:QFN-28-1EP_5x5mm_Pitch0.5mm
- U2: footprint QFN65P400X400X100-16N -> Housings_DFN_QFN:DFN-16-1EP_3x4mm_Pitch0.45mm
- X1: footprint (none) -> Crystals:Crystal_SMD_5032_4Pads
