File: Trx_antena_pcb/Trx_antena_pcb.kicad_pcb (KiCad board)
At the start: 2 copper layers, 41 x 70.5 mm, 14 parts, among them P1 CONN_5, P2 CONN_4

Commit message: "Segundas correcciones. Documentacion"
Parts:
- moved G101 55.6 mm to (87.0, 123.0)
- moved G*** 26.7 mm to (87.2, 94.2)
- moved G*** 3.96 mm to (87.5, 112.2)
Changed lines of the file:
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@@
   (page A4)
   (title_block
-    (title "Poncho Izquierdo - Modelo - Ejemplo - Template")
-    (date "lun 05 oct 2015")
+    (title "Poncho EDU-CIAA-NXP RF 2.4GHz Antena PCB")
+    (date 2016-12-02)
     (rev 1.0)
     (company "Proyecto CIAA - COMPUTADORA INDUSTRIAL ABIERTA ARGENTINA")
     (comment 1 https://github.com/ciaa/Ponchos/tree/master/modelos/doc)
-    (comment 2 "Autores y Licencia del template (Diego Brengi - UNLaM)")
-    (comment 3 "Autor del poncho (COMPLETAR NOMBRE Y APELLIDO). Ver directorio \"doc\"")
-    (comment 4 "CÓDIGO PONCHO:")
+    (comment 2 "Autor y Licencia del template (Diego Brengi - UNLaM)")
+    (comment 3 "Autor y Licencia del poncho (Juan Vicente Montilla-FIUBA). Ver directorio \"doc\"")
+    (comment 4 https://github.com/Juanvmont/Poncho-EDU-CIAA-NXP-RF-2.4GHz-Antena-PCB.git)
   )
   (layers
@@
   )
   (module Poncho_Esqueleto:Logo_EDU-CIAA (layer F.Cu)
-    (at 87.63 116.205)
+    (at 87.5 112.25)
     (fp_text reference G*** (at 0 7.112) (layer F.SilkS) hide
       (effects (font (thickness 0.3048)))
@@
   )
   (module Poncho_Esqueleto:Logo_Poncho (layer F.Cu)
-    (at 100.75 71.25)
+    (at 87.25 94.25)
     (fp_text reference G*** (at 0.127 5.588) (layer F.SilkS) hide
       (effects (font (thickness 0.3)))
@@
   )
   (module Poncho_Esqueleto:Logo_OSHWA (layer F.Cu)
-    (at 68.75 70.5)
+    (at 87 123)
     (fp_text reference G101 (at 0 4.2418) (layer F.SilkS) hide
       (effects (font (size 0.7112 0.4572) (thickness 0.1143)))

Commit message: layout de componentes en pcbnew
Parts:
- removed the REF** at (82.8, 67.5)
- added 1uF/6.3V1: C, Capacitors_SMD:C_0402, F.Cu at (95.0, 122.5)
- added A1: INV_F_ANT, Wpan_Prints:INV_F_ANT, F.Cu at (85.5, 67.8)
- added C1: 100nF, Capacitors_SMD:C_0402, F.Cu at (91.0, 112.0)
- added C10: 1nF, Capacitors_SMD:C_0402, F.Cu at (82.6, 91.5)
- added C11: 1nF, Capacitors_SMD:C_0402, F.Cu at (78.0, 86.7)
- added C12: 1nF, Capacitors_SMD:C_0402, F.Cu at (81.6, 89.3)
- added C13: 1.0pF, Capacitors_SMD:C_0402, F.Cu at (83.8, 82.1)
- added C14: 15pF, Capacitors_SMD:C_0402, F.Cu at (86.1, 84.1)
- added C15: 6.8pF, Capacitors_SMD:C_0402, F.Cu at (84.4, 80.4)
- added C16: 2.7pF, Capacitors_SMD:C_0402, F.Cu at (85.0, 78.4)
- added C2: 100nF, Capacitors_SMD:C_0402, F.Cu at (91.0, 115.0)
- added C3: 100nF, Capacitors_SMD:C_0402, F.Cu at (88.2, 112.5)
- added C4: 100nF, Capacitors_SMD:C_0402, F.Cu at (88.2, 119.2)
- added C5: 100nF, Capacitors_SMD:C_0402, F.Cu at (77.8, 114.0)
- added C6: 100nF, Capacitors_SMD:C_0402, F.Cu at (86.3, 95.7)
- added C7: 100nF, Capacitors_SMD:C_0402, F.Cu at (78.8, 118.5)
- added C8: 100nF, Capacitors_SMD:C_0402, F.Cu at (84.7, 95.7)
- added C9: 2.2uF/4V, Capacitors_SMD:C_0402, F.Cu at (95.0, 89.0)
- added L1: 1K, Capacitors_SMD:C_0402, F.Cu at (94.5, 120.2)
- added L10: 1.0nH, Capacitors_SMD:C_0402, F.Cu at (85.0, 76.9)
- added L2: 1.0nH, Capacitors_SMD:C_0402, F.Cu at (86.8, 93.6)
- added L3: 1.0nH, Capacitors_SMD:C_0402, F.Cu at (84.1, 93.6)
- added L4: 1 K, Capacitors_SMD:C_0402, F.Cu at (95.6, 91.2)
- added L5: 1.0nH, Capacitors_SMD:C_0402, F.Cu at (86.2, 91.4)
- added L6: 2 nF, Capacitors_SMD:C_0402, F.Cu at (84.7, 91.4)
- added L7: 5.1nH, Capacitors_SMD:C_0402, F.Cu at (88.2, 84.6)
- added L8: 1.1nH, Capacitors_SMD:C_0402, F.Cu at (87.6, 82.5)
- added L9: 1.5nH, Capacitors_SMD:C_0402, F.Cu at (84.4, 84.2)
- added R1: 100K, Resistors_SMD:R_0402, F.Cu at (76.2, 120.0)
- added R10: 3.3 1%, Resistors_SMD:R_0402, F.Cu at (83.9, 74.9)
- added R2: 1M, Resistors_SMD:R_0402, F.Cu at (76.2, 123.8)
- added R3: 56K 1%, Resistors_SMD:R_0402, F.Cu at (76.5, 116.0)
- added R4: 0, Resistors_SMD:R_0402, F.Cu at (77.2, 127.2)
- added R5: 0, Resistors_SMD:R_0402, F.Cu at (68.7, 121.5)
- added R6: 0, Resistors_SMD:R_0402, F.Cu at (88.8, 123.5)
- added R7: 0, Resistors_SMD:R_0402, F.Cu at (88.8, 125.5)
- added R8: 330, Resistors_SMD:R_0402, F.Cu at (79.8, 127.2)
- added R9: 4.3k 1%, Resistors_SMD:R_0402, F.Cu at (81.7, 87.7)
- added X1: 32MHz, Crystals:Crystal_SMD_5032_4Pads, F.Cu at (94.2, 114.0)
- U1: renamed from REF**; value QFN-28-1EP_5x5mm_Pitch0.5mm -> CC2520
- U2: renamed from REF**; value DFN-16-1EP_3x4mm_Pitch0.45mm -> CC2591
- moved REF** 22.9 mm to (103.8, 87.5)
- moved REF** 22.6 mm to (103.5, 82.0)
- moved U1 13.8 mm to (83.8, 116.5)
- moved G101 11.9 mm to (95.0, 131.8)
- moved G*** 7.07 mm to (88.5, 105.2)
- moved G*** 1.82 mm to (89.0, 93.8), turned to 90 degrees
- moved U2 1.68 mm to (85.2, 87.8)
Connections:
- U1 pad 1: (no net) -> /Radio/SO
- U1 pad 10: (no net) -> /Radio/GPIO0
- U1 pad 11: (no net) -> Net-(1uF/6.3V1-Pad1)
- U1 pad 12: (no net) -> Net-(C2-Pad1)
- U1 pad 13: (no net) -> Net-(C1-Pad2)
- U1 pad 14: (no net) -> Net-(1uF/6.3V1-Pad1)
- U1 pad 16: (no net) -> Net-(1uF/6.3V1-Pad1)
- U1 pad 17: (no net) -> Net-(C6-Pad1)
- U1 pad 19: (no net) -> Net-(C8-Pad2)
- U1 pad 2: (no net) -> /Radio/SI
- U1 pad 20: (no net) -> Net-(1uF/6.3V1-Pad1)
- U1 pad 22: (no net) -> Net-(1uF/6.3V1-Pad1)
- U1 pad 23: (no net) -> Net-(R3-Pad2)
- U1 pad 24: (no net) -> Net-(1uF/6.3V1-Pad1)
- U1 pad 25: (no net) -> /Radio/RESET
- U1 pad 26: (no net) -> /Radio/VREG_EN
- U1 pad 27: (no net) -> Net-(C7-Pad1)
- U1 pad 28: (no net) -> /Radio/SCLK
- U1 pad 29: (no net) -> GND
- U1 pad 3: (no net) -> GND
- U1 pad 4: (no net) -> /Radio/GPIO5
- U1 pad 5: (no net) -> /Radio/GPIO4
- U1 pad 6: (no net) -> /Radio/GPIO3
- U1 pad 7: (no net) -> /Radio/GPIO2
- U1 pad 8: (no net) -> Net-(1uF/6.3V1-Pad1)
- U1 pad 9: (no net) -> /Radio/GPIO1
- U2 pad 1: (no net) -> /Radio/TL11
- U2 pad 10: (no net) -> /Radio/TL101
- U2 pad 11: (no net) -> Net-(L9-Pad1)
- U2 pad 12: (no net) -> GND
- U2 pad 13: (no net) -> /Radio/TL11
- U2 pad 14: (no net) -> GND
- U2 pad 15: (no net) -> Net-(R9-Pad2)
- U2 pad 16: (no net) -> Net-(C12-Pad2)
- U2 pad 17: (no net) -> GND
- U2 pad 2: (no net) -> Net-(L6-Pad1)
- U2 pad 3: (no net) -> Net-(U2-Pad3)
- U2 pad 4: (no net) -> Net-(L5-Pad2)
- U2 pad 5: (no net) -> /Radio/PAEN
- U2 pad 6: (no net) -> /Radio/EN
- U2 pad 7: (no net) -> /Radio/HGM
- U2 pad 8: (no net) -> GND
- U2 pad 9: (no net) -> GND
- XA1 pad 42: +5VP -> +5V
- XA1 pad 58: Net-(P1-Pad4) -> /Radio/SO
- XA1 pad 60: Net-(P1-Pad2) -> /Radio/SCLK
- XA1 pad 61: Net-(P1-Pad3) -> /Radio/SI
- XA1 pad 69: Net-(XA1-Pad69) -> /Radio/GPIO0
- XA1 pad 71: Net-(XA1-Pad71) -> /Radio/GPIO2
- XA1 pad 72: Net-(P2-Pad4) -> /Radio/GPIO1
- XA1 pad 73: Net-(XA1-Pad73) -> /Radio/GPIO4
- XA1 pad 74: Net-(P2-Pad3) -> /Radio/GPIO3
- XA1 pad 75: Net-(XA1-Pad75) -> /Radio/GPIO6
- XA1 pad 76: Net-(P2-Pad2) -> /Radio/GPIO5
- XA1 pad 78: Net-(XA1-Pad78) -> /Radio/VREG_EN
- XA1 pad 80: Net-(XA1-Pad80) -> /Radio/RESET
Routing:
- net GND: track 67.6 -> 158.8 mm
- net /Radio/GPIO6: track 0.00 -> 32.2 mm
- net /Radio/GPIO5: track 0.00 -> 10.3 mm
- net Net-(P2-Pad2): track 28.0 -> 22.3 mm
- net Net-(P1-Pad2): track 29.1 -> 23.4 mm
- net /Radio/SCLK: track 0.00 -> 5.72 mm
- net Net-(C15-Pad2): track 0.00 -> 5.38 mm
- net Net-(P2-Pad3): track 29.1 -> 24.6 mm
- net Net-(P1-Pad4): track 32.2 -> 27.8 mm
- net /Radio/SO: track 0.00 -> 4.45 mm
- net /Radio/GPIO3: track 0.00 -> 4.45 mm
- net (no net): track 0.00 -> 4.25 mm
- net Net-(C8-Pad1): track 0.00 -> 3.24 mm
- net Net-(C6-Pad2): track 0.00 -> 3.24 mm
- net Net-(P1-Pad3): track 85.3 -> 82.2 mm
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